File: Lignade/AdresseMAC.sch (KiCad schematic (older format))
At the start: 8 parts

Commit message: Remplacement Bus I2C grande distance par Arduino Mini + RS485. Reste : ADC à porter vers module capteur. Renommer nouveaux composants. Vérifier Cablage.
Parts:
- R55, R56, R57, R58, R59, R60, R61, R62: symbol R -> R-RESCUE-Lignade
Changed lines of the file:
@@
-EESchema Schematic File Version 2  date 31/07/2012 18:58:40
+EESchema Schematic File Version 2
+LIBS:Lignade-rescue
 LIBS:power
 LIBS:device
@@
 LIBS:memory
 LIBS:xilinx
-LIBS:special
 LIBS:microcontrollers
 LIBS:dsp
@@
 LIBS:i2c
 LIBS:Lignade-cache
-EELAYER 24  0
+EELAYER 25 0
 EELAYER END
-$Descr A4 11700 8267
+$Descr A4 11693 8268
+encoding utf-8
 Sheet 2 7
 Title ""
@@
 MAC_1
 $Comp
-L R R59
+L R-RESCUE-Lignade R59
 U 1 1 4D96A97D
 P 6900 1850
 F 0 "R59" V 6980 1850 50  0000 C CNN
 F 1 "0R" V 6900 1850 50  0000 C CNN
+F 2 "" H 6900 1850 60  0001 C CNN
+F 3 "" H 6900 1850 60  0001 C CNN
 	1    6900 1850
 	1    0    0    -1
 $EndComp
 $Comp
-L R R60
+L R-RESCUE-Lignade R60
 U 1 1 4D96A97C
 P 6900 2550
 F 0 "R60" V 6980 2550 50  0000 C CNN
 F 1 "0R" V 6900 2550 50  0000 C CNN
+F 2 "" H 6900 2550 60  0001 C CNN
+F 3 "" H 6900 2550 60  0001 C CNN
 	1    6900 2550
 	1    0    0    -1
@@
 F 0 "#PWR03" H 6900 1410 30  0001 C CNN
 F 1 "+3,3V" H 6900 1560 30  0000 C CNN
+F 2 "" H 6900 1450 60  0001 C CNN
+F 3 "" H 6900 1450 60  0001 C CNN
 	1    6900 1450
 	1    0    0    -1
@@
 F 0 "#PWR77" H 6900 2950 40  0001 C CNN
 F 1 "DGND" H 6900 2880 40  0000 C CNN
+F 2 "" H 6900 2950 60  0001 C CNN
+F 3 "" H 6900 2950 60  0001 C CNN
 	1    6900 2950
 	1    0    0    -1
@@
 F 0 "#PWR79" H 6900 4900 40  0001 C CNN
 F 1 "DGND" H 6900 4830 40  0000 C CNN
+F 2 "" H 6900 4900 60  0001 C CNN
+F 3 "" H 6900 4900 60  0001 C CNN
 	1    6900 4900
 	1    0    0    -1
@@
 F 0 "#PWR04" H 6900 3360 30  0001 C CNN
 F 1 "+3,3V" H 6900 3510 30  0000 C CNN
+F 2 "" H 6900 3400 60  0001 C CNN
+F 3 "" H 6900 3400 60  0001 C CNN
 	1    6900 3400
 	1    0    0    -1
 $EndComp
 $Comp
-L R R62
+L R-RESCUE-Lignade R62
 U 1 1 4D96A96E
 P 6900 4500
 F 0 "R62" V 6980 4500 50  0000 C CNN
 F 1 "0R" V 6900 4500 50  0000 C CNN
+F 2 "" H 6900 4500 60  0001 C CNN
+F 3 "" H 6900 4500 60  0001 C CNN
 	1    6900 4500
 	1    0    0    -1
 $EndComp
 $Comp
-L R R61
+L R-RESCUE-Lignade R61
 U 1 1 4D96A96D
 P 6900 3800
 F 0 "R61" V 6980 3800 50  0000 C CNN
 F 1 "0R" V 6900 3800 50  0000 C CNN
+F 2 "" H 6900 3800 60  0001 C CNN
+F 3 "" H 6900 3800 60  0001 C CNN
 	1    6900 3800
 	1    0    0    -1
@@
 MAC_2
 $Comp
-L R R57
+L R-RESCUE-Lignade R57
 U 1 1 4D96A967
 P 4600 3800
 F 0 "R57" V 4680 3800 50  0000 C CNN
 F 1 "0R" V 4600 3800 50  0000 C CNN
+F 2 "" H 4600 3800 60  0001 C CNN
+F 3 "" H 4600 3800 60  0001 C CNN
 	1    4600 3800
 	1    0    0    -1
 $EndComp
 $Comp
-L R R58
+L R-RESCUE-Lignade R58
 U 1 1 4D96A966
 P 4600 4500
 F 0 "R58" V 4680 4500 50  0000 C CNN
 F 1 "0R" V 4600 4500 50  0000 C CNN
+F 2 "" H 4600 4500 60  0001 C CNN
+F 3 "" H 4600 4500 60  0001 C CNN
 	1    4600 4500
 	1    0    0    -1
@@
 F 0 "#PWR05" H 4600 3360 30  0001 C CNN
 F 1 "+3,3V" H 4600 3510 30  0000 C CNN
+F 2 "" H 4600 3400 60  0001 C CNN
+F 3 "" H 4600 3400 60  0001 C CNN
 	1    4600 3400
 	1    0    0    -1
@@
 F 0 "#PWR75" H 4600 4900 40  0001 C CNN
 F 1 "DGND" H 4600 4830 40  0000 C CNN
+F 2 "" H 4600 4900 60  0001 C CNN
+F 3 "" H 4600 4900 60  0001 C CNN
 	1    4600 4900
 	1    0    0    -1
@@
 F 0 "#PWR73" H 4600 2950 40  0001 C CNN
 F 1 "DGND" H 4600 2880 40  0000 C CNN
+F 2 "" H 4600 2950 60  0001 C CNN
+F 3 "" H 4600 2950 60  0001 C CNN
 	1    4600 2950
 	1    0    0    -1
@@
 F 0 "#PWR06" H 4600 1410 30  0001 C CNN
 F 1 "+3,3V" H 4600 1560 30  0000 C CNN
+F 2 "" H 4600 1450 60  0001 C CNN
+F 3 "" H 4600 1450 60  0001 C CNN
 	1    4600 1450
 	1    0    0    -1
 $EndComp
 $Comp
-L R R56
+L R-RESCUE-Lignade R56
 U 1 1 4D96A92E
 P 4600 2550
 F 0 "R56" V 4680 2550 50  0000 C CNN
 F 1 "0R" V 4600 2550 50  0000 C CNN
+F 2 "" H 4600 2550 60  0001 C CNN
+F 3 "" H 4600 2550 60  0001 C CNN
 	1    4600 2550
 	1    0    0    -1
 $EndComp
 $Comp
-L R R55
+L R-RESCUE-Lignade R55
 U 1 1 4D96A928
 P 4600 1850
 F 0 "R55" V 4680 1850 50  0000 C CNN
 F 1 "0R" V 4600 1850 50  0000 C CNN
+F 2 "" H 4600 1850 60  0001 C CNN
+F 3 "" H 4600 1850 60  0001 C CNN
 	1    4600 1850
 	1    0    0    -1
