File: Lignade/Connects.sch (KiCad schematic (older format))
At the start: 20 parts

Commit message: Remplacement Bus I2C grande distance par Arduino Mini + RS485. Reste : ADC à porter vers module capteur. Renommer nouveaux composants. Vérifier Cablage.
Parts:
- R63, R64, R65, R66, R67, R68, R69, R70: symbol R -> R-RESCUE-Lignade
Changed lines of the file:
@@
-EESchema Schematic File Version 2  date 31/07/2012 18:58:40
+EESchema Schematic File Version 2
+LIBS:Lignade-rescue
 LIBS:power
 LIBS:device
@@
 LIBS:memory
 LIBS:xilinx
-LIBS:special
 LIBS:microcontrollers
 LIBS:dsp
@@
 LIBS:i2c
 LIBS:Lignade-cache
-EELAYER 24  0
+EELAYER 25 0
 EELAYER END
-$Descr A4 11700 8267
+$Descr A4 11693 8268
+encoding utf-8
 Sheet 3 7
 Title ""
@@
 Strap Alim1
 $Comp
-L R R67
+L R-RESCUE-Lignade R67
 U 1 1 4DB13D4E
 P 6850 5300
 F 0 "R67" V 6930 5300 50  0000 C CNN
 F 1 "0R" V 6850 5300 50  0000 C CNN
+F 2 "" H 6850 5300 60  0001 C CNN
+F 3 "" H 6850 5300 60  0001 C CNN
 	1    6850 5300
 	1    0    0    -1
 $EndComp
 $Comp
-L R R70
+L R-RESCUE-Lignade R70
 U 1 1 4DB13D49
 P 9650 4850
 F 0 "R70" V 9730 4850 50  0000 C CNN
 F 1 "0R" V 9650 4850 50  0000 C CNN
+F 2 "" H 9650 4850 60  0001 C CNN
+F 3 "" H 9650 4850 60  0001 C CNN
 	1    9650 4850
 	1    0    0    -1
 $EndComp
 $Comp
-L R R69
+L R-RESCUE-Lignade R69
 U 1 1 4DB13D47
 P 8900 5300
 F 0 "R69" V 8980 5300 50  0000 C CNN
 F 1 "0R" V 8900 5300 50  0000 C CNN
+F 2 "" H 8900 5300 60  0001 C CNN
+F 3 "" H 8900 5300 60  0001 C CNN
 	1    8900 5300
 	1    0    0    -1
 $EndComp
 $Comp
-L R R68
+L R-RESCUE-Lignade R68
 U 1 1 4DB13D42
 P 7650 4850
 F 0 "R68" V 7730 4850 50  0000 C CNN
 F 1 "0R" V 7650 4850 50  0000 C CNN
+F 2 "" H 7650 4850 60  0001 C CNN
+F 3 "" H 7650 4850 60  0001 C CNN
 	1    7650 4850
 	1    0    0    -1
 $EndComp
 $Comp
-L R R66
+L R-RESCUE-Lignade R66
 U 1 1 4DB13D3A
 P 5600 4850
 F 0 "R66" V 5680 4850 50  0000 C CNN
 F 1 "0R" V 5600 4850 50  0000 C CNN
+F 2 "" H 5600 4850 60  0001 C CNN
+F 3 "" H 5600 4850 60  0001 C CNN
 	1    5600 4850
 	1    0    0    -1
 $EndComp
 $Comp
-L R R65
+L R-RESCUE-Lignade R65
 U 1 1 4DB13D28
 P 4800 5300
 F 0 "R65" V 4880 5300 50  0000 C CNN
 F 1 "0R" V 4800 5300 50  0000 C CNN
+F 2 "" H 4800 5300 60  0001 C CNN
+F 3 "" H 4800 5300 60  0001 C CNN
 	1    4800 5300
 	1    0    0    -1
 $EndComp
 $Comp
-L R R64
+L R-RESCUE-Lignade R64
 U 1 1 4DB13D21
 P 3550 4850
 F 0 "R64" V 3630 4850 50  0000 C CNN
 F 1 "0R" V 3550 4850 50  0000 C CNN
+F 2 "" H 3550 4850 60  0001 C CNN
+F 3 "" H 3550 4850 60  0001 C CNN
 	1    3550 4850
 	1    0    0    -1
 $EndComp
 $Comp
-L R R63
+L R-RESCUE-Lignade R63
 U 1 1 4DB13D1B
 P 2750 5300
 F 0 "R63" V 2830 5300 50  0000 C CNN
 F 1 "0R" V 2750 5300 50  0000 C CNN
+F 2 "" H 2750 5300 60  0001 C CNN
+F 3 "" H 2750 5300 60  0001 C CNN
 	1    2750 5300
 	1    0    0    -1
@@
 F 0 "#PWR61" H 3650 7100 40  0001 C CNN
 F 1 "DGND" H 3650 7030 40  0000 C CNN
+F 2 "" H 3650 7100 60  0001 C CNN
+F 3 "" H 3650 7100 60  0001 C CNN
 	1    3650 7100
 	1    0    0    -1
@@
 F 0 "#PWR64" H 5700 7100 40  0001 C CNN
 F 1 "DGND" H 5700 7030 40  0000 C CNN
+F 2 "" H 5700 7100 60  0001 C CNN
+F 3 "" H 5700 7100 60  0001 C CNN
 	1    5700 7100
 	1    0    0    -1
@@
 F 0 "#PWR67" H 7800 7100 40  0001 C CNN
 F 1 "DGND" H 7800 7030 40  0000 C CNN
+F 2 "" H 7800 7100 60  0001 C CNN
+F 3 "" H 7800 7100 60  0001 C CNN
 	1    7800 7100
 	1    0    0    -1
@@
 F 0 "#PWR69" H 9800 7100 40  0001 C CNN
 F 1 "DGND" H 9800 7030 40  0000 C CNN
+F 2 "" H 9800 7100 60  0001 C CNN
+F 3 "" H 9800 7100 60  0001 C CNN
 	1    9800 7100
 	1    0    0    -1
@@
 F 0 "#PWR71" H 10550 5700 40  0001 C CNN
 F 1 "DGND" H 10550 5630 40  0000 C CNN
+F 2 "" H 10550 5700 60  0001 C CNN
+F 3 "" H 10550 5700 60  0001 C CNN
 	1    10550 5700
 	1    0    0    -1
@@
 F 0 "#PWR68" H 8550 5700 40  0001 C CNN
 F 1 "DGND" H 8550 5630 40  0000 C CNN
+F 2 "" H 8550 5700 60  0001 C CNN
+F 3 "" H 8550 5700 60  0001 C CNN
 	1    8550 5700
 	1    0    0    -1
@@
 F 0 "#PWR65" H 6500 5700 40  0001 C CNN
 F 1 "DGND" H 6500 5630 40  0000 C CNN
+F 2 "" H 6500 5700 60  0001 C CNN
+F 3 "" H 6500 5700 60  0001 C CNN
 	1    6500 5700
 	1    0    0    -1
@@
 F 0 "#PWR62" H 4450 5700 40  0001 C CNN
 F 1 "DGND" H 4450 5630 40  0000 C CNN
+F 2 "" H 4450 5700 60  0001 C CNN
+F 3 "" H 4450 5700 60  0001 C CNN
 	1    4450 5700
 	1    0    0    -1
@@
 F 0 "#PWR70" H 10250 1850 40  0001 C CNN
 F 1 "DGND" H 10250 1780 40  0000 C CNN
+F 2 "" H 10250 1850 60  0001 C CNN
+F 3 "" H 10250 1850 60  0001 C CNN
 	1    10250 1850
 	1    0    0    -1
@@
 F 0 "#PWR66" H 7800 1850 40  0001 C CNN
 F 1 "DGND" H 7800 1780 40  0000 C CNN
+F 2 "" H 7800 1850 60  0001 C CNN
+F 3 "" H 7800 1850 60  0001 C CNN
 	1    7800 1850
 	1    0    0    -1
@@
 F 0 "#PWR63" H 5250 1850 40  0001 C CNN
 F 1 "DGND" H 5250 1780 40  0000 C CNN
+F 2 "" H 5250 1850 60  0001 C CNN
+F 3 "" H 5250 1850 60  0001 C CNN
 	1    5250 1850
 	1    0    0    -1
@@
 F 0 "#PWR60" H 2750 1850 40  0001 C CNN
 F 1 "DGND" H 2750 1780 40  0000 C CNN
+F 2 "" H 2750 1850 60  0001 C CNN
+F 3 "" H 2750 1850 60  0001 C CNN
 	1    2750 1850
 	1    0    0    -1
@@
 F 0 "CONN3" H 3600 6900 60  0000 C CNN
 F 1 "RJ45_1PORT" V 3850 6400 60  0000 C CNN
+F 2 "" H 3450 6450 60  0001 C CNN
+F 3 "" H 3450 6450 60  0001 C CNN
 	1    3450 6450
 	1    0    0    -1
@@
 F 0 "CONN4" H 4400 5500 60  0000 C CNN
 F 1 "RJ45_1PORT" V 4650 5000 60  0000 C CNN
+F 2 "" H 4250 5050 60  0001 C CNN
+F 3 "" H 4250 5050 60  0001 C CNN
 	1    4250 5050
 	1    0    0    -1
@@
 F 0 "CONN6" H 5650 6900 60  0000 C CNN
 F 1 "RJ45_1PORT" V 5900 6400 60  0000 C CNN
+F 2 "" H 5500 6450 60  0001 C CNN
+F 3 "" H 5500 6450 60  0001 C CNN
 	1    5500 6450
 	1    0    0    -1
@@
 F 0 "CONN7" H 6450 5500 60  0000 C CNN
 F 1 "RJ45_1PORT" V 6700 5000 60  0000 C CNN
+F 2 "" H 6300 5050 60  0001 C CNN
+F 3 "" H 6300 5050 60  0001 C CNN
 	1    6300 5050
 	1    0    0    -1
@@
 F 0 "CONN10" H 8500 5500 60  0000 C CNN
 F 1 "RJ45_1PORT" V 8750 5000 60  0000 C CNN
+F 2 "" H 8350 5050 60  0001 C CNN
+F 3 "" H 8350 5050 60  0001 C CNN
 	1    8350 5050
 	1    0    0    -1
@@
 F 0 "CONN9" H 7750 6900 60  0000 C CNN
 F 1 "RJ45_1PORT" V 8000 6400 60  0000 C CNN
+F 2 "" H 7600 6450 60  0001 C CNN
+F 3 "" H 7600 6450 60  0001 C CNN
 	1    7600 6450
 	1    0    0    -1
@@
 F 0 "CONN11" H 9750 6900 60  0000 C CNN
 F 1 "RJ45_1PORT" V 10000 6400 60  0000 C CNN
+F 2 "" H 9600 6450 60  0001 C CNN
+F 3 "" H 9600 6450 60  0001 C CNN
 	1    9600 6450
 	1    0    0    -1
@@
 F 0 "CONN13" H 10500 5500 60  0000 C CNN
 F 1 "RJ45_1PORT" V 10750 5000 60  0000 C CNN
+F 2 "" H 10350 5050 60  0001 C CNN
+F 3 "" H 10350 5050 60  0001 C CNN
 	1    10350 5050
 	1    0    0    -1
@@
 F 0 "CONN12" H 10200 1650 60  0000 C CNN
 F 1 "RJ45_1PORT" V 10450 1150 60  0000 C CNN
+F 2 "" H 10050 1200 60  0001 C CNN
+F 3 "" H 10050 1200 60  0001 C CNN
 	1    10050 1200
 	1    0    0    -1
@@
 F 0 "CONN8" H 7750 1650 60  0000 C CNN
 F 1 "RJ45_1PORT" V 8000 1150 60  0000 C CNN
+F 2 "" H 7600 1200 60  0001 C CNN
+F 3 "" H 7600 1200 60  0001 C CNN
 	1    7600 1200
 	1    0    0    -1
@@
 F 0 "CONN5" H 5200 1650 60  0000 C CNN
 F 1 "RJ45_1PORT" V 5450 1150 60  0000 C CNN
+F 2 "" H 5050 1200 60  0001 C CNN
+F 3 "" H 5050 1200 60  0001 C CNN
 	1    5050 1200
 	1    0    0    -1
@@
 F 0 "CONN2" H 2700 1650 60  0000 C CNN
 F 1 "RJ45_1PORT" V 2950 1150 60  0000 C CNN
+F 2 "" H 2550 1200 60  0001 C CNN
+F 3 "" H 2550 1200 60  0001 C CNN
 	1    2550 1200
 	1    0    0    -1
