File: Lignade/I_O_Relays.sch (KiCad schematic (older format))
At the start: 44 parts, among them P17 CONN_1, P18 CONN_1, P19 CONN_1, P20 CONN_1, P21 CONN_1, P22 CONN_1, P23 CONN_1, P24 CONN_1, Q1 PNP, Q2 PNP, Q3 PNP, Q4 PNP, Q5 PNP, Q6 PNP, Q7 PNP, Q8 PNP, U4 74LVC132, U5 74LVC132

Commit message: Remplacement Bus I2C grande distance par Arduino Mini + RS485. Reste : ADC à porter vers module capteur. Renommer nouveaux composants. Vérifier Cablage.
Parts:
- C2, C3: symbol C -> C-RESCUE-Lignade
- Q1, Q2, Q3, Q4, Q5, Q6, Q7, Q8: symbol PNP -> PNP-RESCUE-Lignade
- R27, R28, R29, R30, R31, R32, R33, R34, R35, R36, R37, R38, R39, R40, R41, R42, R43, R44, R45, R46, R47, R48, R49, R50: symbol R -> R-RESCUE-Lignade
