File: Lignade/Lignade.sch (KiCad schematic (older format))
At the start: 37 parts, among them K1 CONN_3, P1 CONN_1, P2 CONN_1, P3 CONN_1, P4 CONN_1, P5 CONN_1, P6 CONN_1, P7 CONN_1, P8 CONN_1

Commit message: Remplacement Bus I2C grande distance par Arduino Mini + RS485. Reste : ADC à porter vers module capteur. Renommer nouveaux composants. Vérifier Cablage.
Parts:
- CONN1: symbol CONN-HIROSE-132_PTS -> CONN-HIROSE-132_pts
- R1, R10, R11, R12, R13, R14, R15, R16, R17, R18, R19, R2, R20, R21, R22, R23, R24, R25, R26, R3, R4, R5, R6, R7, R71, R8, R9: symbol R -> R-RESCUE-Lignade
Changed lines of the file:
@@
-EESchema Schematic File Version 2  date 31/07/2012 18:58:40
+EESchema Schematic File Version 2
+LIBS:Lignade-rescue
 LIBS:power
 LIBS:device
@@
 LIBS:memory
 LIBS:xilinx
-LIBS:special
 LIBS:microcontrollers
 LIBS:dsp
@@
 LIBS:i2c
 LIBS:Lignade-cache
-EELAYER 24  0
+EELAYER 25 0
 EELAYER END
-$Descr A4 11700 8267
+$Descr A4 11693 8268
+encoding utf-8
 Sheet 1 7
 Title ""
@@
 RD7
 $Comp
-L R R71
+L R-RESCUE-Lignade R71
 U 1 1 4DB15D37
 P 4300 2250
 F 0 "R71" V 4300 2300 50  0000 C CNN
 F 1 "0R" V 4300 2150 50  0000 C CNN
+F 2 "" H 4300 2250 60  0001 C CNN
+F 3 "" H 4300 2250 60  0001 C CNN
 	1    4300 2250
 	0    1    1    0
@@
 F 0 "#PWR01" H 4950 1040 20  0001 C CNN
 F 1 "+5V" H 4950 1040 30  0000 C CNN
+F 2 "" H 4950 950 60  0001 C CNN
+F 3 "" H 4950 950 60  0001 C CNN
 	1    4950 950
 	1    0    0    -1
 $EndComp
 $Comp
-L R R24
+L R-RESCUE-Lignade R24
 U 1 1 4DAE63F4
 P 5000 1350
 F 0 "R24" V 5000 1400 50  0000 C CNN
 F 1 "0R" V 5000 1250 50  0000 C CNN
+F 2 "" H 5000 1350 60  0001 C CNN
+F 3 "" H 5000 1350 60  0001 C CNN
 	1    5000 1350
 	0    1    1    0
 $EndComp
 $Comp
-L R R25
+L R-RESCUE-Lignade R25
 U 1 1 4DAE63EE
 P 5000 1450
 F 0 "R25" V 5000 1500 50  0000 C CNN
 F 1 "0R" V 5000 1350 50  0000 C CNN
+F 2 "" H 5000 1450 60  0001 C CNN
+F 3 "" H 5000 1450 60  0001 C CNN
 	1    5000 1450
 	0    1    1    0
 $EndComp
 $Comp
-L R R26
+L R-RESCUE-Lignade R26
 U 1 1 4DAE63E2
 P 5000 1550
 F 0 "R26" V 5000 1600 50  0000 C CNN
 F 1 "0R" V 5000 1450 50  0000 C CNN
+F 2 "" H 5000 1550 60  0001 C CNN
+F 3 "" H 5000 1550 60  0001 C CNN
 	1    5000 1550
 	0    1    1    0
@@
 F 0 "#PWR2" H 3000 7700 40  0001 C CNN
 F 1 "DGND" H 3000 7630 40  0000 C CNN
+F 2 "" H 3000 7700 60  0001 C CNN
+F 3 "" H 3000 7700 60  0001 C CNN
 	1    3000 7700
 	1    0    0    -1
@@
 F 0 "K1" V 5500 7000 50  0000 C CNN
 F 1 "CONN_3" V 5600 7000 40  0000 C CNN
+F 2 "" H 5550 7000 60  0001 C CNN
+F 3 "" H 5550 7000 60  0001 C CNN
 	1    5550 7000
 	-1   0    0    -1
 $EndComp
 $Comp
-L CONN-HIROSE-132_PTS CONN1
+L CONN-HIROSE-132_pts CONN1
 U 1 1 4D70492F
 P 3150 4050
 F 0 "CONN1" H 2700 7300 60  0000 C CNN
 F 1 "CONN-HIROSE-132_PTS" H 3150 7150 60  0000 C CNN
+F 2 "" H 3150 4050 60  0001 C CNN
+F 3 "" H 3150 4050 60  0001 C CNN
 	1    3150 4050
 	1    0    0    -1
@@
 F 0 "P1" H 1080 1450 40  0000 L CNN
 F 1 "CONN_1" H 1000 1505 30  0001 C CNN
+F 2 "" H 1000 1450 60  0001 C CNN
+F 3 "" H 1000 1450 60  0001 C CNN
 	1    1000 1450
 	-1   0    0    -1
@@
 F 0 "P2" H 1080 1550 40  0000 L CNN
 F 1 "CONN_1" H 1000 1605 30  0001 C CNN
+F 2 "" H 1000 1550 60  0001 C CNN
+F 3 "" H 1000 1550 60  0001 C CNN
 	1    1000 1550
 	-1   0    0    -1
@@
 F 0 "P3" H 1080 1650 40  0000 L CNN
 F 1 "CONN_1" H 1000 1705 30  0001 C CNN
+F 2 "" H 1000 1650 60  0001 C CNN
+F 3 "" H 1000 1650 60  0001 C CNN
 	1    1000 1650
 	-1   0    0    -1
@@
 F 0 "P4" H 1080 1750 40  0000 L CNN
 F 1 "CONN_1" H 1000 1805 30  0001 C CNN
+F 2 "" H 1000 1750 60  0001 C CNN
+F 3 "" H 1000 1750 60  0001 C CNN
 	1    1000 1750
 	-1   0    0    -1
@@
 F 0 "P5" H 1080 1850 40  0000 L CNN
 F 1 "CONN_1" H 1000 1905 30  0001 C CNN
+F 2 "" H 1000 1850 60  0001 C CNN
+F 3 "" H 1000 1850 60  0001 C CNN
 	1    1000 1850
 	-1   0    0    -1
@@
 F 0 "P6" H 1080 1950 40  0000 L CNN
 F 1 "CONN_1" H 1000 2005 30  0001 C CNN
+F 2 "" H 1000 1950 60  0001 C CNN
+F 3 "" H 1000 1950 60  0001 C CNN
 	1    1000 1950
 	-1   0    0    -1
@@
 F 0 "P7" H 1080 2050 40  0000 L CNN
 F 1 "CONN_1" H 1000 2105 30  0001 C CNN
+F 2 "" H 1000 2050 60  0001 C CNN
+F 3 "" H 1000 2050 60  0001 C CNN
 	1    1000 2050
 	-1   0    0    -1
@@
 F 0 "P8" H 1080 2150 40  0000 L CNN
 F 1 "CONN_1" H 1000 2205 30  0001 C CNN
+F 2 "" H 1000 2150 60  0001 C CNN
+F 3 "" H 1000 2150 60  0001 C CNN
 	1    1000 2150
 	-1   0    0    1
 $EndComp
 $Comp
-L R R1
+L R-RESCUE-Lignade R1
 U 1 1 4D6D96A4
 P 1900 4350
 F 0 "R1" V 1900 4400 50  0000 C CNN
 F 1 "0R" V 1900 4250 50  0000 C CNN
+F 2 "" H 1900 4350 60  0001 C CNN
+F 3 "" H 1900 4350 60  0001 C CNN
 	1    1900 4350
 	0    1    1    0
 $EndComp
 $Comp
-L R R2
+L R-RESCUE-Lignade R2
 U 1 1 4D6D96A1
 P 1900 4450
 F 0 "R2" V 1900 4500 50  0000 C CNN
 F 1 "0R" V 1900 4350 50  0000 C CNN
+F 2 "" H 1900 4450 60  0001 C CNN
+F 3 "" H 1900 4450 60  0001 C CNN
 	1    1900 4450
 	0    1    1    0
 $EndComp
 $Comp
-L R R3
+L R-RESCUE-Lignade R3
 U 1 1 4D6D969D
 P 1900 5650
 F 0 "R3" V 1900 5700 50  0000 C CNN
 F 1 "0R" V 1900 5550 50  0000 C CNN
+F 2 "" H 1900 5650 60  0001 C CNN
+F 3 "" H 1900 5650 60  0001 C CNN
 	1    1900 5650
 	0    1    1    0
 $EndComp
 $Comp
-L R R4
+L R-RESCUE-Lignade R4
 U 1 1 4D6D969A
 P 1900 5750
 F 0 "R4" V 1900 5800 50  0000 C CNN
 F 1 "0R" V 1900 5650 50  0000 C CNN
+F 2 "" H 1900 5750 60  0001 C CNN
+F 3 "" H 1900 5750 60  0001 C CNN
 	1    1900 5750
 	0    1    1    0
 $EndComp
 $Comp
-L R R5
+L R-RESCUE-Lignade R5
 U 1 1 4D6D9697
 P 1900 5850
 F 0 "R5" V 1900 5900 50  0000 C CNN
 F 1 "0R" V 1900 5750 50  0000 C CNN
+F 2 "" H 1900 5850 60  0001 C CNN
+F 3 "" H 1900 5850 60  0001 C CNN
 	1    1900 5850
 	0    1    1    0
 $EndComp
 $Comp
-L R R6
+L R-RESCUE-Lignade R6
 U 1 1 4D6D9693
 P 1900 5950
 F 0 "R6" V 1900 6000 50  0000 C CNN
 F 1 "0R" V 1900 5850 50  0000 C CNN
+F 2 "" H 1900 5950 60  0001 C CNN
+F 3 "" H 1900 5950 60  0001 C CNN
 	1    1900 5950
 	0    1    1    0
 $EndComp
 $Comp
-L R R7
+L R-RESCUE-Lignade R7
 U 1 1 4D6D968F
 P 1900 6850
 F 0 "R7" V 1900 6900 50  0000 C CNN
 F 1 "0R" V 1900 6750 50  0000 C CNN
+F 2 "" H 1900 6850 60  0001 C CNN
+F 3 "" H 1900 6850 60  0001 C CNN
 	1    1900 6850
 	0    1    1    0
 $EndComp
 $Comp
-L R R8
+L R-RESCUE-Lignade R8
 U 1 1 4D6D9685
 P 1900 6950
 F 0 "R8" V 1900 7000 50  0000 C CNN
 F 1 "0R" V 1900 6850 50  0000 C CNN
+F 2 "" H 1900 6950 60  0001 C CNN
+F 3 "" H 1900 6950 60  0001 C CNN
 	1    1900 6950
 	0    1    1    0
 $EndComp
 $Comp
-L R R23
+L R-RESCUE-Lignade R23
 U 1 1 4D6D963B
 P 4300 7050
 F 0 "R23" V 4300 7100 50  0000 C CNN
 F 1 "0R" V 4300 6950 50  0000 C CNN
+F 2 "" H 4300 7050 60  0001 C CNN
+F 3 "" H 4300 7050 60  0001 C CNN
 	1    4300 7050
 	0    1    1    0
 $EndComp
 $Comp
-L R R22
+L R-RESCUE-Lignade R22
 U 1 1 4D6D9634
 P 4300 6850
 F 0 "R22" V 4300 6900 50  0000 C CNN
 F 1 "0R" V 4300 6750 50  0000 C CNN
+F 2 "" H 4300 6850 60  0001 C CNN
+F 3 "" H 4300 6850 60  0001 C CNN
 	1    4300 6850
 	0    1    1    0
 $EndComp
 $Comp
-L R R21
+L R-RESCUE-Lignade R21
 U 1 1 4D6D95D6
 P 4300 4350
 F 0 "R21" V 4300 4400 50  0000 C CNN
 F 1 "0R" V 4300 4250 50  0000 C CNN
+F 2 "" H 4300 4350 60  0001 C CNN
+F 3 "" H 4300 4350 60  0001 C CNN
 	1    4300 4350
 	0    1    1    0
 $EndComp
 $Comp
-L R R20
+L R-RESCUE-Lignade R20
 U 1 1 4D6D95D2
 P 4300 4250
 F 0 "R20" V 4300 4300 50  0000 C CNN
 F 1 "0R" V 4300 4150 50  0000 C CNN
+F 2 "" H 4300 4250 60  0001 C CNN
+F 3 "" H 4300 4250 60  0001 C CNN
 	1    4300 4250
 	0    1    1    0
 $EndComp
 $Comp
-L R R19
+L R-RESCUE-Lignade R19
 U 1 1 4D6D95CE
 P 4300 4150
 F 0 "R19" V 4300 4200 50  0000 C CNN
 F 1 "0R" V 4300 4050 50  0000 C CNN
+F 2 "" H 4300 4150 60  0001 C CNN
+F 3 "" H 4300 4150 60  0001 C CNN
 	1    4300 4150
 	0    1    1    0
 $EndComp
 $Comp
-L R R18
+L R-RESCUE-Lignade R18
 U 1 1 4D6D95CA
 P 4300 4050
 F 0 "R18" V 4300 4100 50  0000 C CNN
 F 1 "0R" V 4300 3950 50  0000 C CNN
+F 2 "" H 4300 4050 60  0001 C CNN
+F 3 "" H 4300 4050 60  0001 C CNN
 	1    4300 4050
 	0    1    1    0
 $EndComp
 $Comp
-L R R17
+L R-RESCUE-Lignade R17
 U 1 1 4D6D95C5
 P 4300 3950
 F 0 "R17" V 4300 4000 50  0000 C CNN
 F 1 "0R" V 4300 3850 50  0000 C CNN
+F 2 "" H 4300 3950 60  0001 C CNN
+F 3 "" H 4300 3950 60  0001 C CNN
 	1    4300 3950
 	0    1    1    0
 $EndComp
 $Comp
-L R R16
+L R-RESCUE-Lignade R16
 U 1 1 4D6D95BC
 P 4300 3850
 F 0 "R16" V 4300 3900 50  0000 C CNN
 F 1 "0R" V 4300 3750 50  0000 C CNN
+F 2 "" H 4300 3850 60  0001 C CNN
+F 3 "" H 4300 3850 60  0001 C CNN
 	1    4300 3850
 	0    1    1    0
 $EndComp
 $Comp
-L R R9
+L R-RESCUE-Lignade R9
 U 1 1 4D6D9527
 P 1950 2250
 F 0 "R9" V 1950 2300 50  0000 C CNN
 F 1 "0R" V 1950 2150 50  0000 C CNN
+F 2 "" H 1950 2250 60  0001 C CNN
+F 3 "" H 1950 2250 60  0001 C CNN
 	1    1950 2250
 	0    1    1    0
 $EndComp
 $Comp
-L R R15
+L R-RESCUE-Lignade R15
 U 1 1 4D6D951F
 P 4300 3150
 F 0 "R15" V 4300 3200 50  0000 C CNN
 F 1 "0R" V 4300 3050 50  0000 C CNN
+F 2 "" H 4300 3150 60  0001 C CNN
+F 3 "" H 4300 3150 60  0001 C CNN
 	1    4300 3150
 	0    1    1    0
 $EndComp
 $Comp
-L R R14
+L R-RESCUE-Lignade R14
 U 1 1 4D6D951C
 P 4300 3050
 F 0 "R14" V 4300 3100 50  0000 C CNN
 F 1 "0R" V 4300 2950 50  0000 C CNN
+F 2 "" H 4300 3050 60  0001 C CNN
+F 3 "" H 4300 3050 60  0001 C CNN
 	1    4300 3050
 	0    1    1    0
 $EndComp
 $Comp
-L R R13
+L R-RESCUE-Lignade R13
 U 1 1 4D6D9519
 P 4300 2950
 F 0 "R13" V 4300 3000 50  0000 C CNN
 F 1 "0R" V 4300 2850 50  0000 C CNN
+F 2 "" H 4300 2950 60  0001 C CNN
+F 3 "" H 4300 2950 60  0001 C CNN
 	1    4300 2950
 	0    1    1    0
 $EndComp
 $Comp
-L R R12
+L R-RESCUE-Lignade R12
 U 1 1 4D6D9514
 P 4300 2850
 F 0 "R12" V 4300 2900 50  0000 C CNN
 F 1 "0R" V 4300 2750 50  0000 C CNN
+F 2 "" H 4300 2850 60  0001 C CNN
+F 3 "" H 4300 2850 60  0001 C CNN
 	1    4300 2850
 	0    1    1    0
 $EndComp
 $Comp
-L R R11
+L R-RESCUE-Lignade R11
 U 1 1 4D6D950B
 P 4300 2750
 F 0 "R11" V 4300 2800 50  0000 C CNN
 F 1 "0R" V 4300 2650 50  0000 C CNN
+F 2 "" H 4300 2750 60  0001 C CNN
+F 3 "" H 4300 2750 60  0001 C CNN
 	1    4300 2750
 	0    1    1    0
 $EndComp
 $Comp
-L R R10
+L R-RESCUE-Lignade R10
 U 1 1 4D6D94B4
 P 4300 2150
 F 0 "R10" V 4300 2200 50  0000 C CNN
 F 1 "0R" V 4300 2050 50  0000 C CNN
+F 2 "" H 4300 2150 60  0001 C CNN
+F 3 "" H 4300 2150 60  0001 C CNN
 	1    4300 2150
 	0    1    1    0
@@
 F 0 "#PWR02" H 600 910 30  0001 C CNN
 F 1 "+3.3V" H 600 1060 30  0000 C CNN
+F 2 "" H 600 950 60  0001 C CNN
+F 3 "" H 600 950 60  0001 C CNN
 	1    600  950
 	1    0    0    -1
