File: Lignade/LignadeAlims.sch (KiCad schematic (older format))
At the start: 24 parts, among them P25 CONN_1, P26 CONN_1, P27 CONN_1, U6 LM1117, U7 LM1117, U8 TC1262-3.3V

Commit message: Remplacement Bus I2C grande distance par Arduino Mini + RS485. Reste : ADC à porter vers module capteur. Renommer nouveaux composants. Vérifier Cablage.
Parts:
- C10, C11, C12, C4, C5, C6, C7, C8, C9: symbol C -> C-RESCUE-Lignade
- R51, R52, R53, R54: symbol R -> R-RESCUE-Lignade
