File: Lignade/LignadeI2C.sch (KiCad schematic (older format))
At the start: 22 parts, among them K2 RELAY_1RT, K3 RELAY_1RT, K4 RELAY_1RT, K5 RELAY_1RT, K6 RELAY_1RT, K7 RELAY_1RT, K8 RELAY_1RT, K9 RELAY_1RT, M1 MODULE_I2C, P10 CONN_1, P11 CONN_1, P12 CONN_1, P13 CONN_1, P14 CONN_1, P15 CONN_1, P16 CONN_1, P9 CONN_1, U1 DS3680, U2 DS3680, U3 74HCT138

Commit message: Remplacement Bus I2C grande distance par Arduino Mini + RS485. Reste : ADC à porter vers module capteur. Renommer nouveaux composants. Vérifier Cablage.
Parts:
- C1: symbol C -> C-RESCUE-Lignade
- R?: symbol R -> R-RESCUE-Lignade
Changed lines of the file:
@@
-EESchema Schematic File Version 2  date 31/07/2012 18:58:40
+EESchema Schematic File Version 2
+LIBS:Lignade-rescue
 LIBS:power
 LIBS:device
@@
 LIBS:memory
 LIBS:xilinx
-LIBS:special
 LIBS:microcontrollers
 LIBS:dsp
@@
 LIBS:i2c
 LIBS:Lignade-cache
-EELAYER 24  0
+EELAYER 25 0
 EELAYER END
-$Descr A4 11700 8267
+$Descr A4 11693 8268
+encoding utf-8
 Sheet 7 7
 Title ""
@@
 	6000 1700 6150 1700
 $Comp
-L R R?
+L R-RESCUE-Lignade R?
 U 1 1 50180E6B
 P 5750 1700
 F 0 "R?" V 5830 1700 50  0000 C CNN
 F 1 "R" V 5750 1700 50  0000 C CNN
+F 2 "" H 5750 1700 60  0001 C CNN
+F 3 "" H 5750 1700 60  0001 C CNN
 	1    5750 1700
 	0    1    1    0
@@
 F 0 "U3" H 6700 1700 60  0000 C CNN
 F 1 "74HCT138" H 6750 1550 60  0000 C CNN
+F 2 "" H 6750 1600 60  0001 C CNN
+F 3 "" H 6750 1600 60  0001 C CNN
 	1    6750 1600
 	1    0    0    -1
@@
 F 0 "#PWR037" H 6750 890 20  0001 C CNN
 F 1 "+5V" H 6750 890 30  0000 C CNN
+F 2 "" H 6750 800 60  0001 C CNN
+F 3 "" H 6750 800 60  0001 C CNN
 	1    6750 800
 	1    0    0    -1
@@
 F 0 "#PWR038" H 5400 1690 20  0001 C CNN
 F 1 "+5V" H 5400 1690 30  0000 C CNN
+F 2 "" H 5400 1600 60  0001 C CNN
+F 3 "" H 5400 1600 60  0001 C CNN
 	1    5400 1600
 	1    0    0    -1
@@
 F 0 "#PWR16" H 7550 1000 40  0001 C CNN
 F 1 "DGND" H 7550 930 40  0000 C CNN
+F 2 "" H 7550 1000 60  0001 C CNN
+F 3 "" H 7550 1000 60  0001 C CNN
 	1    7550 1000
 	1    0    0    -1
 $EndComp
 $Comp
-L C C1
+L C-RESCUE-Lignade C1
 U 1 1 4DAE59A8
 P 7050 950
+AR Path="/4DAE59A8" Ref="C1"  Part="1"
+AR Path="/4D6C87F2/4DAE59A8" Ref="C1"  Part="1"
 F 0 "C1" H 7100 1050 50  0000 L CNN
 F 1 "100nF" H 7100 850 50  0000 L CNN
+F 2 "" H 7050 950 60  0001 C CNN
+F 3 "" H 7050 950 60  0001 C CNN
 	1    7050 950
 	0    1    1    0
@@
 F 0 "#PWR15" H 6750 2300 40  0001 C CNN
 F 1 "DGND" H 6750 2230 40  0000 C CNN
+F 2 "" H 6750 2300 60  0001 C CNN
+F 3 "" H 6750 2300 60  0001 C CNN
 	1    6750 2300
 	1    0    0    -1
@@
 F 0 "P16" H 1280 6050 40  0000 L CNN
 F 1 "CONN_1" H 1200 6105 30  0001 C CNN
+F 2 "" H 1200 6050 60  0001 C CNN
+F 3 "" H 1200 6050 60  0001 C CNN
 	1    1200 6050
 	1    0    0    -1
@@
 F 0 "#PWR7" H 2500 7500 40  0001 C CNN
 F 1 "DGND" H 2500 7430 40  0000 C CNN
+F 2 "" H 2500 7500 60  0001 C CNN
+F 3 "" H 2500 7500 60  0001 C CNN
 	1    2500 7500
 	1    0    0    -1
@@
 F 0 "#PWR6" H 1250 2650 40  0001 C CNN
 F 1 "DGND" H 1250 2580 40  0000 C CNN
+F 2 "" H 1250 2650 60  0001 C CNN
+F 3 "" H 1250 2650 60  0001 C CNN
 	1    1250 2650
 	1    0    0    -1
@@
 F 0 "#PWR8" H 3850 1200 40  0001 C CNN
 F 1 "DGND" H 3850 1130 40  0000 C CNN
+F 2 "" H 3850 1200 60  0001 C CNN
+F 3 "" H 3850 1200 60  0001 C CNN
 	1    3850 1200
 	1    0    0    -1
@@
 F 0 "M1" H 2450 1650 60  0000 C CNN
 F 1 "MODULE_I2C" V 2450 2350 60  0000 C CNN
+F 2 "" H 2600 2000 60  0001 C CNN
+F 3 "" H 2600 2000 60  0001 C CNN
 	1    2600 2000
 	1    0    0    -1
@@
 F 0 "K9" H 7550 4750 70  0000 C CNN
 F 1 "RELAY_1RT" H 7800 4350 70  0000 C CNN
+F 2 "" H 7800 4500 60  0001 C CNN
+F 3 "" H 7800 4500 60  0001 C CNN
 	1    7800 4500
 	1    0    0    -1
@@
 F 0 "#PWR039" H 8500 4250 20  0001 C CNN
 F 1 "+12V" H 8500 4400 30  0000 C CNN
+F 2 "" H 8500 4300 60  0001 C CNN
+F 3 "" H 8500 4300 60  0001 C CNN
 	1    8500 4300
 	1    0    0    -1
@@
 F 0 "#PWR040" H 1250 1250 20  0001 C CNN
 F 1 "+12V" H 1250 1400 30  0000 C CNN
+F 2 "" H 1250 1300 60  0001 C CNN
+F 3 "" H 1250 1300 60  0001 C CNN
 	1    1250 1300
 	-1   0    0    -1
@@
 F 0 "#PWR041" H 6250 4650 20  0001 C CNN
 F 1 "+12V" H 6250 4800 30  0000 C CNN
+F 2 "" H 6250 4700 60  0001 C CNN
+F 3 "" H 6250 4700 60  0001 C CNN
 	1    6250 4700
 	1    0    0    -1
@@
 F 0 "K5" H 5300 5150 70  0000 C CNN
 F 1 "RELAY_1RT" H 5550 4750 70  0000 C CNN
+F 2 "" H 5550 4900 60  0001 C CNN
+F 3 "" H 5550 4900 60  0001 C CNN
 	1    5550 4900
 	1    0    0    -1
@@
 F 0 "#PWR042" H 8500 5650 20  0001 C CNN
 F 1 "+12V" H 8500 5800 30  0000 C CNN
+F 2 "" H 8500 5700 60  0001 C CNN
+F 3 "" H 8500 5700 60  0001 C CNN
 	1    8500 5700
 	1    0    0    -1
@@
 F 0 "K8" H 7550 6150 70  0000 C CNN
 F 1 "RELAY_1RT" H 7800 5750 70  0000 C CNN
+F 2 "" H 7800 5900 60  0001 C CNN
+F 3 "" H 7800 5900 60  0001 C CNN
 	1    7800 5900
 	1    0    0    -1
@@
 F 0 "K4" H 5300 5850 70  0000 C CNN
 F 1 "RELAY_1RT" H 5550 5450 70  0000 C CNN
+F 2 "" H 5550 5600 60  0001 C CNN
+F 3 "" H 5550 5600 60  0001 C CNN
 	1    5550 5600
 	1    0    0    -1
@@
 F 0 "#PWR043" H 6250 5350 20  0001 C CNN
 F 1 "+12V" H 6250 5500 30  0000 C CNN
+F 2 "" H 6250 5400 60  0001 C CNN
+F 3 "" H 6250 5400 60  0001 C CNN
 	1    6250 5400
 	1    0    0    -1
@@
 F 0 "K7" H 5300 4450 70  0000 C CNN
 F 1 "RELAY_1RT" H 5550 4050 70  0000 C CNN
+F 2 "" H 5550 4200 60  0001 C CNN
+F 3 "" H 5550 4200 60  0001 C CNN
 	1    5550 4200
 	1    0    0    -1
@@
 F 0 "#PWR044" H 6250 3950 20  0001 C CNN
 F 1 "+12V" H 6250 4100 30  0000 C CNN
+F 2 "" H 6250 4000 60  0001 C CNN
+F 3 "" H 6250 4000 60  0001 C CNN
 	1    6250 4000
 	1    0    0    -1
@@
 F 0 "#PWR045" H 8500 4950 20  0001 C CNN
 F 1 "+12V" H 8500 5100 30  0000 C CNN
+F 2 "" H 8500 5000 60  0001 C CNN
+F 3 "" H 8500 5000 60  0001 C CNN
 	1    8500 5000
 	1    0    0    -1
@@
 F 0 "K3" H 7550 5450 70  0000 C CNN
 F 1 "RELAY_1RT" H 7800 5050 70  0000 C CNN
+F 2 "" H 7800 5200 60  0001 C CNN
+F 3 "" H 7800 5200 60  0001 C CNN
 	1    7800 5200
 	1    0    0    -1
@@
 F 0 "K6" H 7550 7050 70  0000 C CNN
 F 1 "RELAY_1RT" H 7800 6650 70  0000 C CNN
+F 2 "" H 7800 6800 60  0001 C CNN
+F 3 "" H 7800 6800 60  0001 C CNN
 	1    7800 6800
 	1    0    0    -1
@@
 F 0 "#PWR046" H 8500 6550 20  0001 C CNN
 F 1 "+12V" H 8500 6700 30  0000 C CNN
+F 2 "" H 8500 6600 60  0001 C CNN
+F 3 "" H 8500 6600 60  0001 C CNN
 	1    8500 6600
 	1    0    0    -1
@@
 F 0 "#PWR047" H 6250 6050 20  0001 C CNN
 F 1 "+12V" H 6250 6200 30  0000 C CNN
+F 2 "" H 6250 6100 60  0001 C CNN
+F 3 "" H 6250 6100 60  0001 C CNN
 	1    6250 6100
 	1    0    0    -1
@@
 F 0 "K2" H 5300 6550 70  0000 C CNN
 F 1 "RELAY_1RT" H 5550 6150 70  0000 C CNN
+F 2 "" H 5550 6300 60  0001 C CNN
+F 3 "" H 5550 6300 60  0001 C CNN
 	1    5550 6300
 	1    0    0    -1
@@
 F 0 "U2" H 3350 7000 60  0000 C CNN
 F 1 "DS3680" H 3000 7000 60  0000 C CNN
+F 2 "" H 3250 6450 60  0001 C CNN
+F 3 "" H 3250 6450 60  0001 C CNN
 	1    3250 6450
 	1    0    0    -1
@@
 F 0 "U1" H 3350 5050 60  0000 C CNN
 F 1 "DS3680" H 3000 5050 60  0000 C CNN
+F 2 "" H 3250 4500 60  0001 C CNN
+F 3 "" H 3250 4500 60  0001 C CNN
 	1    3250 4500
 	1    0    0    -1
@@
 F 0 "#PWR048" H 1250 1140 20  0001 C CNN
 F 1 "+5V" H 1250 1140 30  0000 C CNN
+F 2 "" H 1250 1050 60  0001 C CNN
+F 3 "" H 1250 1050 60  0001 C CNN
 	1    1250 1050
 	-1   0    0    -1
@@
 F 0 "P15" H 1280 5850 40  0000 L CNN
 F 1 "CONN_1" H 1200 5905 30  0001 C CNN
+F 2 "" H 1200 5850 60  0001 C CNN
+F 3 "" H 1200 5850 60  0001 C CNN
 	1    1200 5850
 	1    0    0    -1
@@
 F 0 "P14" H 1280 5650 40  0000 L CNN
 F 1 "CONN_1" H 1200 5705 30  0001 C CNN
+F 2 "" H 1200 5650 60  0001 C CNN
+F 3 "" H 1200 5650 60  0001 C CNN
 	1    1200 5650
 	1    0    0    -1
@@
 F 0 "P13" H 1280 5450 40  0000 L CNN
 F 1 "CONN_1" H 1200 5505 30  0001 C CNN
+F 2 "" H 1200 5450 60  0001 C CNN
+F 3 "" H 1200 5450 60  0001 C CNN
 	1    1200 5450
 	1    0    0    -1
@@
 F 0 "P12" H 1280 5250 40  0000 L CNN
 F 1 "CONN_1" H 1200 5305 30  0001 C CNN
+F 2 "" H 1200 5250 60  0001 C CNN
+F 3 "" H 1200 5250 60  0001 C CNN
 	1    1200 5250
 	1    0    0    -1
@@
 F 0 "P11" H 1280 5050 40  0000 L CNN
 F 1 "CONN_1" H 1200 5105 30  0001 C CNN
+F 2 "" H 1200 5050 60  0001 C CNN
+F 3 "" H 1200 5050 60  0001 C CNN
 	1    1200 5050
 	1    0    0    -1
@@
 F 0 "P10" H 1280 4850 40  0000 L CNN
 F 1 "CONN_1" H 1200 4905 30  0001 C CNN
+F 2 "" H 1200 4850 60  0001 C CNN
+F 3 "" H 1200 4850 60  0001 C CNN
 	1    1200 4850
 	1    0    0    -1
@@
 F 0 "P9" H 1280 4650 40  0000 L CNN
 F 1 "CONN_1" H 1200 4705 30  0001 C CNN
+F 2 "" H 1200 4650 60  0001 C CNN
+F 3 "" H 1200 4650 60  0001 C CNN
 	1    1200 4650
 	1    0    0    -1
