File: Lignade/Satellite.sch (KiCad schematic (older format))
At the start: 13 parts, among them K5 CONN_3, P1 CONN_3, P2 CONN_3, P3 CONN_3, P4 CONN_3, P5 CONN_2, P6 CONN_2, P7 CONN_2, P8 CONN_2

Commit message: Remplacement Bus I2C grande distance par Arduino Mini + RS485. Reste : ADC à porter vers module capteur. Renommer nouveaux composants. Vérifier Cablage.
Parts:
- removed R1, R24: 0R, symbol R
- added C? (x2): C, symbol C
- added CONN?: RJ45_1PORT, symbol RJ45_1PORT
- added L? (x2): L_Small, symbol L_Small
- added R? (x4): R, symbol R
- R21: symbol R -> R-RESCUE-Satellite
Connections:
- net labels removed: SEL_I2C
- wire segments 48 -> 81
Other:
- moved on the sheet: CONN1, K5, P1, P2, P3, P4, P5, P6, P7, P8, R21
