File: Lignade/SatelliteAlim.sch (KiCad schematic (older format))
At the start: 26 parts, among them P10 CONN_1, P11 CONN_1, P23 CONN_1, P9 CONN_1, U1 LM1117, U2 TC1262-3.3V, U8 LM1117

Commit message: Remplacement Bus I2C grande distance par Arduino Mini + RS485. Reste : ADC à porter vers module capteur. Renommer nouveaux composants. Vérifier Cablage.
Parts:
- C1, C13, C14, C2, C3, C4, C5, C6, C7: symbol C -> C-RESCUE-Satellite
- R2, R3, R4, R5: symbol R -> R-RESCUE-Satellite
