File: Lignade/Satellite_Capteurs.sch (KiCad schematic (older format))
At the start: 6 parts, among them M2 MODULE_CAPTEUR, U5 24LC512, U6 PCA9538D

Commit message: Remplacement Bus I2C grande distance par Arduino Mini + RS485. Reste : ADC à porter vers module capteur. Renommer nouveaux composants. Vérifier Cablage.
Parts:
- C10, C11: symbol C -> C-RESCUE-Satellite
- R20: symbol R -> R-RESCUE-Satellite
Connections:
- net labels removed: SELECT
- wire segments 52 -> 49
Changed lines of the file:
@@
-EESchema Schematic File Version 2  date mar. 10 mai 2011 21:09:00 ICT
+EESchema Schematic File Version 2
+LIBS:Satellite-rescue
 LIBS:power
 LIBS:device
@@
 LIBS:memory
 LIBS:xilinx
-LIBS:special
 LIBS:microcontrollers
 LIBS:dsp
@@
 LIBS:Lignade
 LIBS:i2c
+LIBS:ok-ic-com
+LIBS:shield_arduino
 LIBS:Satellite-cache
-EELAYER 24  0
+EELAYER 25 0
 EELAYER END
-$Descr A4 11700 8267
+$Descr A4 11693 8268
+encoding utf-8
 Sheet 4 6
 Title ""
@@
 	3000 1400 2900 1400
 Wire Wire Line
-	5600 1900 5700 1900
-Wire Wire Line
 	2900 1350 2900 1500
 Connection ~ 5100 800
@@
 	2900 2450 2900 2350
 Wire Wire Line
-	2400 2150 2050 2150
-Wire Wire Line
 	3400 1400 3450 1400
 Wire Wire Line
@@
 	4200 650  4200 4250
 Connection ~ 4200 650
-Wire Wire Line
-	4050 4800 4200 4800
 Wire Wire Line
 	4850 5450 4850 5700
@@
 F 0 "#PWR08" H 5550 2110 30  0001 C CNN
 F 1 "+3.3V" H 5550 2260 30  0000 C CNN
+F 2 "" H 5550 2150 60  0001 C CNN
+F 3 "" H 5550 2150 60  0001 C CNN
 	1    5550 2150
 	1    0    0    -1
@@
 F 0 "U6" H 6100 2100 60  0000 C CNN
 F 1 "PCA9538D" H 6450 2650 60  0000 C CNN
+F 2 "" H 6100 2100 60  0001 C CNN
+F 3 "" H 6100 2100 60  0001 C CNN
 	1    6100 2100
 	1    0    0    -1
@@
 F 0 "#PWR09" H 5200 5700 40  0001 C CNN
 F 1 "AGND" H 5200 5630 50  0000 C CNN
+F 2 "" H 5200 5700 60  0001 C CNN
+F 3 "" H 5200 5700 60  0001 C CNN
 	1    5200 5700
 	1    0    0    -1
@@
 F 0 "#PWR53" H 4850 5700 40  0001 C CNN
 F 1 "DGND" H 4850 5630 40  0000 C CNN
+F 2 "" H 4850 5700 60  0001 C CNN
+F 3 "" H 4850 5700 60  0001 C CNN
 	1    4850 5700
 	1    0    0    -1
@@
 F 0 "#PWR010" H 5050 3510 30  0001 C CNN
 F 1 "+3.3V" H 5050 3660 30  0000 C CNN
+F 2 "" H 5050 3550 60  0001 C CNN
+F 3 "" H 5050 3550 60  0001 C CNN
 	1    5050 3550
 	1    0    0    -1
 $EndComp
-Text GLabel 4050 4800 0    60   Output ~ 0
-SELECT
 $Comp
 L MODULE_CAPTEUR M2
@@
 F 0 "M2" H 4550 5000 60  0000 C CNN
 F 1 "MODULE_CAPTEUR" H 5000 4450 60  0000 C CNN
+F 2 "" H 5000 4450 60  0001 C CNN
+F 3 "" H 5000 4450 60  0001 C CNN
 	1    5000 4450
 	1    0    0    -1
 $EndComp
-Text GLabel 2050 2150 0    60   Output ~ 0
-SELECT
-Text GLabel 5600 1900 0    60   Output ~ 0
-SELECT
 $Comp
 L DGND #PWR46
@@
 F 0 "#PWR46" H 1800 2000 40  0001 C CNN
 F 1 "DGND" H 1800 1930 40  0000 C CNN
+F 2 "" H 1800 2000 60  0001 C CNN
+F 3 "" H 1800 2000 60  0001 C CNN
 	1    1800 2000
 	1    0    0    -1
@@
 F 0 "#PWR48" H 5400 2200 40  0001 C CNN
 F 1 "DGND" H 5400 2130 40  0000 C CNN
+F 2 "" H 5400 2200 60  0001 C CNN
+F 3 "" H 5400 2200 60  0001 C CNN
 	1    5400 2200
 	1    0    0    -1
@@
 F 0 "#PWR45" H 5650 1550 40  0001 C CNN
 F 1 "DGND" H 5650 1480 40  0000 C CNN
+F 2 "" H 5650 1550 60  0001 C CNN
+F 3 "" H 5650 1550 60  0001 C CNN
 	1    5650 1550
 	1    0    0    -1
@@
 F 0 "#PWR51" H 6100 2750 40  0001 C CNN
 F 1 "DGND" H 6100 2680 40  0000 C CNN
+F 2 "" H 6100 2750 60  0001 C CNN
+F 3 "" H 6100 2750 60  0001 C CNN
 	1    6100 2750
 	1    0    0    -1
@@
 F 0 "#PWR50" H 3500 2450 40  0001 C CNN
 F 1 "DGND" H 3500 2380 40  0000 C CNN
+F 2 "" H 3500 2450 60  0001 C CNN
+F 3 "" H 3500 2450 60  0001 C CNN
 	1    3500 2450
 	1    0    0    -1
@@
 F 0 "#PWR44" H 3450 1500 40  0001 C CNN
 F 1 "DGND" H 3450 1430 40  0000 C CNN
+F 2 "" H 3450 1500 60  0001 C CNN
+F 3 "" H 3450 1500 60  0001 C CNN
 	1    3450 1500
 	1    0    0    -1
@@
 F 0 "#PWR49" H 2900 2450 40  0001 C CNN
 F 1 "DGND" H 2900 2380 40  0000 C CNN
+F 2 "" H 2900 2450 60  0001 C CNN
+F 3 "" H 2900 2450 60  0001 C CNN
 	1    2900 2450
 	1    0    0    -1
 $EndComp
 $Comp
-L R R20
+L R-RESCUE-Satellite R20
 U 1 1 4D774027
 P 5350 1350
 F 0 "R20" V 5430 1350 50  0000 C CNN
 F 1 "1K" V 5350 1350 50  0000 C CNN
+F 2 "" H 5350 1350 60  0001 C CNN
+F 3 "" H 5350 1350 60  0001 C CNN
 	1    5350 1350
 	1    0    0    -1
@@
 F 0 "#PWR011" H 5350 1010 30  0001 C CNN
 F 1 "+3.3V" H 5450 1100 30  0000 C CNN
+F 2 "" H 5350 1050 60  0001 C CNN
+F 3 "" H 5350 1050 60  0001 C CNN
 	1    5350 1050
 	1    0    0    -1
@@
 AD:0x70/0x71\n
 $Comp
-L C C10
+L C-RESCUE-Satellite C10
 U 1 1 4D74FCCA
 P 3200 1400
+AR Path="/4D74FCCA" Ref="C10"  Part="1"
+AR Path="/4D74F960/4D74FCCA" Ref="C10"  Part="1"
 F 0 "C10" H 3250 1500 50  0000 L CNN
 F 1 "100nF" H 3250 1300 50  0000 L CNN
+F 2 "" H 3200 1400 60  0001 C CNN
+F 3 "" H 3200 1400 60  0001 C CNN
 	1    3200 1400
 	0    1    1    0
 $EndComp
 $Comp
-L C C11
+L C-RESCUE-Satellite C11
 U 1 1 4D74FCC0
 P 5850 1450
+AR Path="/4D74FCC0" Ref="C11"  Part="1"
+AR Path="/4D74F960/4D74FCC0" Ref="C11"  Part="1"
 F 0 "C11" H 5900 1550 50  0000 L CNN
 F 1 "100nF" H 5900 1350 50  0000 L CNN
+F 2 "" H 5850 1450 60  0001 C CNN
+F 3 "" H 5850 1450 60  0001 C CNN
 	1    5850 1450
 	0    -1   -1   0
@@
 F 0 "#PWR012" H 6100 1360 30  0001 C CNN
 F 1 "+3.3V" H 6100 1510 30  0000 C CNN
+F 2 "" H 6100 1400 60  0001 C CNN
+F 3 "" H 6100 1400 60  0001 C CNN
 	1    6100 1400
 	1    0    0    -1
@@
 F 0 "#PWR013" H 2900 1310 30  0001 C CNN
 F 1 "+3.3V" H 2900 1460 30  0000 C CNN
+F 2 "" H 2900 1350 60  0001 C CNN
+F 3 "" H 2900 1350 60  0001 C CNN
 	1    2900 1350
 	1    0    0    -1
@@
 F 0 "U5" H 3200 2150 60  0000 C CNN
 F 1 "24LC512" H 2600 2350 60  0000 C CNN
+F 2 "" H 2900 1950 60  0001 C CNN
+F 3 "" H 2900 1950 60  0001 C CNN
 	1    2900 1950
 	1    0    0    -1
