File: Lignade/Satellite_IO.sch (KiCad schematic (older format))
At the start: 32 parts, among them P12 CONN_1, P13 CONN_1, P14 CONN_1, P15 CONN_1, P16 CONN_1, P17 CONN_1, P18 CONN_1, Q1 PNP, Q2 PNP, Q3 PNP, Q4 PNP, U3 74LVC132, U4 74LVC132

Commit message: Remplacement Bus I2C grande distance par Arduino Mini + RS485. Reste : ADC à porter vers module capteur. Renommer nouveaux composants. Vérifier Cablage.
Parts:
- C12, C8, C9: symbol C -> C-RESCUE-Satellite
- Q1, Q2, Q3, Q4: symbol PNP -> PNP-RESCUE-Satellite
- R10, R11, R13, R14, R15, R16, R17, R18, R19, R25, R26, R27, R6, R7, R8, R9: symbol R -> R-RESCUE-Satellite
